File: wemos-br1-board.brd (EAGLE design)
At the start: 58.4 x 40.6 mm, 29 parts, among them J1 2p-2.54, J2 3p-2.54, U1 PHOTORESISTOR-5528-10K

Commit message: board fab version
Parts:
- moved R5 0.63 mm to (53.3, 48.9)
- moved R6 0.63 mm to (58.4, 48.9)
Routing:
- net 5V: track 119.3 -> 122.8 mm
- net 3V3: track 137.8 -> 138.7 mm
- net D2: track 43.1 -> 43.9 mm
- net LED_OUT: track 39.8 -> 40.3 mm
